File: pcb/alarmclock.kicad_pcb (KiCad board)
At the start: 2 copper layers, 22 parts, among them J1 Conn_01x06_Male, J2 Conn_01x02_Female, J3 Conn_01x02_Female, J4 Conn_01x05_Female, J5 Conn_01x08_Male, Q1 BC547, U1 DS1307+, U2 DHT11, Y1 32.7kHz

Commit message: updates
Parts:
- removed J2: Conn_01x02_Female, Pin_Headers:Pin_Header_Straight_1x02_Pitch2.54mm
- removed RV1: 10K, Potentiometers:Potentiometer_Alps_RK097_Single_Vertical
- added BT1: CR2032, Battery_Holders:Keystone_1058_1x2032-CoinCell, F.Cu at (113.0, 127.0)
- added BT2: 6V, Pin_Headers:Pin_Header_Straight_1x02_Pitch1.27mm, F.Cu at (63.5, 67.3)
- added BZ1: Buzzer, Buzzers_Beepers:Buzzer_12x9.5RM7.6, F.Cu at (156.2, 123.2)
- added D2: D, Diodes_THT:D_5W_P10.16mm_Horizontal, F.Cu at (67.3, 69.8)
- added Q2: BC547, TO_SOT_Packages_THT:TO-92_Molded_Narrow, F.Cu at (63.5, 76.2)
- added Q3: BC547, TO_SOT_Packages_THT:TO-92_Molded_Narrow, F.Cu at (67.3, 113.0)
- added R11: 10K, Resistors_THT:R_Axial_DIN0516_L15.5mm_D5.0mm_P25.40mm_Horizontal, F.Cu at (154.3, 92.7)
- added SW1: SW_Push, Buttons_Switches_THT:SW_PUSH_6mm, F.Cu at (115.6, 95.2)
- added U3: MCP23017, SMD_Packages:SOIC-28, B.Cu at (131.4, 81.9)
- D1: value 3.3V -> 2.7V
- R2: value 1K -> 120
- R3: value 10K -> 1K
- moved J1 33.1 mm to (137.2, 61.0)
Connections:
- D1 pad 1: Z_OUT -> 3.3V
- D1 pad 2: VSS -> Net-(D1-Pad2)
- J1 pad 2: VDD -> (no net)
- J1 pad 3: VSS -> (no net)
- J3 pad 1: +BATT -> (no net)
- J3 pad 2: VSS -> GND
- J5 pad 1: Z_OUT -> 3.3V
- J5 pad 2: VSS -> GND
- J5 pad 8: LED -> (no net)
- MCU1 pad 1: VDD -> 5.5V
- MCU1 pad 10: VSS -> BUZZER
- MCU1 pad 12: VSS -> GND
- MCU1 pad 17: VSS -> GND
- MCU1 pad 20: VSS -> GND
- Q1 pad 1: Net-(Q1-Pad1) -> 3.3V
- Q1 pad 3: LED -> GND
- R10 pad 1: VDD -> 5.5V
- R2 pad 1: Z_OUT -> 3.3V
- R2 pad 2: VDD -> 6V
- R3 pad 1: MCLR -> Net-(Q3-Pad2)
- R3 pad 2: VDD -> BUZZER
- R4 pad 1: VDD -> 5.5V
- R5 pad 1: VDD -> 5.5V
- R6 pad 1: VDD -> 5.5V
- R7 pad 1: VDD -> 5.5V
- R8 pad 1: VDD -> 5.5V
- R9 pad 1: VDD -> 5.5V
- U1 pad 3: +BATT -> Net-(BT1-Pad1)
- U1 pad 4: VSS -> GND
- U1 pad 7: Net-(U1-Pad7) -> (no net)
- U1 pad 8: VDD -> 5.5V
- U2 pad 1: VDD -> 5.5V
- U2 pad 4: VSS -> GND
Other:
- board outline added: 152.4 x 113.7 mm
